File: hardware/kicad/analog_rails.kicad_sch (KiCad schematic)
At the start: 43 parts, among them U10 LMR62014XMF, U11 LM27761DSG, U12 REF5025AID, U13 LT3042EMSE, U9 803 type, 3.08 V

Commit message: feat(hardware): draw decisions D-95, D-97 and D-98
The three decisions that follow the circuit simulations and need no
copper are drawn in the schematic and on the board as changes of
values, part numbers, fitted flags and texts:

- D-95: C32, C33 and C34 of the rail monitor are 10 nF C0G
  (GRM1885C1H103JA01D), not 1 nF.
- D-98: the damper on the input from the controller module is fitted,
  R14 at 0.33 ohm (ERJ-6RQFR33V) and C5 at 10 uF (CL21A106KAYNNNE).
- D-97: the position U9 stays without a part, and its text no longer
  names the detector with the time-out of 0.24 s.

No track, via, zone or footprint position changed. The electrical
rules check and the design rules check with schematic parity report
nothing. The bill of materials (151 lines for 370 parts), the
schematic PDF, the pictures of the three sheets and the two renderings
of the board are exported again.

D-96, the position for a capacitor at U28, is not drawn: it needs a
footprint and copper.
Parts:
- U9: value 803 type, 3.08 V -> Detector, ms time-out
Other:
- note added: "U10: VOUT = 1.23 V x (1 + R32 / R33) = 13.5 V, 1.6 MHz; not gated by 5V_OK. C25 closes the switching loop at D6; C27 is 7 uF at 13.5 V (datasheet curve). U9: position for an open-drain voltage detector at the enable pin of U10, not fitted. U10 has no soft start; as drawn it starts in one go from the current-limited input (simulated; bench test open). The 803 type, time-out 0.24 s, is no longer th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"
- note removed: "U10: VOUT = 1.23 V x (1 + R32 / R33) = 13.5 V, 1.6 MHz; not gated by 5V_OK. C25 closes the switching loop at D6; C27 is 7 uF at 13.5 V (datasheet curve). U9: position for an open-drain voltage detector of the 803 type (3.08 V), not fitted. With it the converter stays off while +5V is below that level. Fit it if U10, which has no soft start, does not start from the current-limited input (bench)."
Changed lines of the file:
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@@
 		(comment 1 "+13.5 V boost, +12 V_A, -4 V_A and the 2.5 V reference")
 	)
-	(text "U10: VOUT = 1.23 V x (1 + R32 / R33) = 13.5 V, 1.6 MHz;\nnot gated by 5V_OK. C25 closes the switching loop at D6;\nC27 is 7 uF at 13.5 V (datasheet curve).\nU9: position for an open-drain voltage detector of the 803 type\n(3.08 V), not fitted. With it the converter stays off while +5V is\nbelow that level. Fit it if U10, which has no soft start, does not\nstart from the current-limited input (bench)."
+	(text "U10: VOUT = 1.23 V x (1 + R32 / R33) = 13.5 V, 1.6 MHz;\nnot gated by 5V_OK. C25 closes the switching loop at D6;\nC27 is 7 uF at 13.5 V (datasheet curve).\nU9: position for an open-drain voltage detector at the enable pin\nof U10, not fitted. U10 has no soft start; as drawn it starts in\none go from the current-limited input (simulated; bench test open).\nThe 803 type, time-out 0.24 s, is no longer the part meant: a\nremedy, if the bench asks for one, has a time-out of milliseconds."
 		(exclude_from_sim no)
 		(at 116.84 60.96 0)
@@
 			)
 		)
-		(property "Value" "803 type, 3.08 V"
+		(property "Value" "Detector, ms time-out"
 			(at 41.91 71.12 0)
 			(show_name no)
