File: hardware/kicad/power_input.kicad_sch (KiCad schematic)
At the start: 40 parts, among them J2 USB-C power, U2 TPD4E1U06DBVR, U3 TPS259621DDAR, U4 TPS259621DDAR, U5 TPS2116DRLR

Commit message: feat(hardware): draw decisions D-95, D-97 and D-98
The three decisions that follow the circuit simulations and need no
copper are drawn in the schematic and on the board as changes of
values, part numbers, fitted flags and texts:

- D-95: C32, C33 and C34 of the rail monitor are 10 nF C0G
  (GRM1885C1H103JA01D), not 1 nF.
- D-98: the damper on the input from the controller module is fitted,
  R14 at 0.33 ohm (ERJ-6RQFR33V) and C5 at 10 uF (CL21A106KAYNNNE).
- D-97: the position U9 stays without a part, and its text no longer
  names the detector with the time-out of 0.24 s.

No track, via, zone or footprint position changed. The electrical
rules check and the design rules check with schematic parity report
nothing. The bill of materials (151 lines for 370 parts), the
schematic PDF, the pictures of the three sheets and the two renderings
of the board are exported again.

D-96, the position for a capacitor at U28, is not drawn: it needs a
footprint and copper.
Parts:
- C5: value 10u 25V -> 10u 25V X5R; MPN (none) -> CL21A106KAYNNNE; Manufacturer (none) -> Samsung Electro-Mechanics; now fitted; now in the parts list
- R14: value 0.33R -> 0.33R 1%; MPN (none) -> ERJ-6RQFR33V; Manufacturer (none) -> Panasonic; now fitted; now in the parts list
Other:
- note added: "U3 (eFuse B) does the same for the supply from the USB connector of the controller module: same thresholds (R5, R6), limit 0.76 A (0.67 A to 0.85 A, R13), fastest ramp, turn-on delay about 0.08 ms typical. R17 defines VBUS_P while U3 is off. R14 and C5 (0.33 ohm, 10 uF) damp VBUS_P when the data cable is plugged again while USB-C feeds +5V: without them VBUS_P reaches 5.94 V (simulated); U5 is ra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"
- note removed: "U3 (eFuse B) does the same for the supply from the USB connector of the controller module: same thresholds (R5, R6), limit 0.76 A (0.67 A to 0.85 A, R13), fastest ramp, turn-on delay about 0.08 ms typical. R17 defines VBUS_P while U3 is off. R14, C5: position for a damper of VBUS_P, not fitted. Fit 0.33 ohm and 10 uF if the bench shows VBUS_P above 6.0 V when the data cable is plugged again. U5 d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"
Changed lines of the file:
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@@
 		(comment 1 "Two USB inputs, one eFuse each, joined by a priority multiplexer that drives +5V")
 	)
-	(text "U3 (eFuse B) does the same for the supply from the USB connector of the controller\nmodule: same thresholds (R5, R6), limit 0.76 A (0.67 A to 0.85 A, R13), fastest ramp,\nturn-on delay about 0.08 ms typical. R17 defines VBUS_P while U3 is off.\nR14, C5: position for a damper of VBUS_P, not fitted. Fit 0.33 ohm and 10 uF if the\nbench shows VBUS_P above 6.0 V when the data cable is plugged again.\nU5 drives +5V from USB-C (VBUS_CP) while PR1 is above 1.0 V, that is while VBUS_CP is\nabove 2.37 V (2.15 V to 2.59 V, calculated from R18, R19), otherwise from the module\n(VBUS_P). It blocks reverse current into both inputs. C8 delays PR1 by 0.19 ms, until\nthe ramp of U4 is nearly complete.\nOrder of the thresholds on a falling rail: supervisor of +5V 3.83 V to 4.00 V (next\nsheet), eFuse off 2.67 V to 2.87 V, change of source 2.15 V to 2.59 V. The multiplexer\nleaves USB-C only when U4 is already off.\nSRC_ST (TP5): open = USB-C in use, low = supply of the module in use."
+	(text "U3 (eFuse B) does the same for the supply from the USB connector of the controller\nmodule: same thresholds (R5, R6), limit 0.76 A (0.67 A to 0.85 A, R13), fastest ramp,\nturn-on delay about 0.08 ms typical. R17 defines VBUS_P while U3 is off.\nR14 and C5 (0.33 ohm, 10 uF) damp VBUS_P when the data cable is plugged again while USB-C\nfeeds +5V: without them VBUS_P reaches 5.94 V (simulated); U5 is rated 6.0 V (datasheet).\nU5 drives +5V from USB-C (VBUS_CP) while PR1 is above 1.0 V, that is while VBUS_CP is\nabove 2.37 V (2.15 V to 2.59 V, calculated from R18, R19), otherwise from the module\n(VBUS_P). It blocks reverse current into both inputs. C8 delays PR1 by 0.19 ms, until\nthe ramp of U4 is nearly complete.\nOrder of the thresholds on a falling rail: supervisor of +5V 3.83 V to 4.00 V (next\nsheet), eFuse off 2.67 V to 2.87 V, change of source 2.15 V to 2.59 V. The multiplexer\nleaves USB-C only when U4 is already off.\nSRC_ST (TP5): open = USB-C in use, low = supply of the module in use."
 		(exclude_from_sim no)
 		(at 162.56 15.24 0)
@@
 		(body_style 1)
 		(exclude_from_sim no)
-		(in_bom no)
+		(in_bom yes)
 		(on_board yes)
 		(in_pos_files yes)
-		(dnp yes)
+		(dnp no)
 		(property "Reference" "C5"
 			(at 167.892 161.81 0)
@@
 			)
 		)
-		(property "Value" "10u 25V"
+		(property "Value" "10u 25V X5R"
 			(at 167.892 163.61 0)
 			(show_name no)
@@
 			)
 		)
+		(property "MPN" "CL21A106KAYNNNE"
+			(at 165.1 162.56 0)
+			(hide yes)
+			(show_name no)
+			(do_not_autoplace no)
+			(effects
+				(font
+					(size 1.27 1.27)
+				)
+			)
+		)
+		(property "Manufacturer" "Samsung Electro-Mechanics"
+			(at 165.1 162.56 0)
+			(hide yes)
+			(show_name no)
+			(do_not_autoplace no)
+			(effects
+				(font
+					(size 1.27 1.27)
+				)
+			)
+		)
 		(pin "1"
 		)
@@
 		(body_style 1)
 		(exclude_from_sim no)
-		(in_bom no)
+		(in_bom yes)
 		(on_board yes)
 		(in_pos_files yes)
-		(dnp yes)
+		(dnp no)
 		(property "Reference" "R14"
 			(at 166.876 150.38 0)
@@
 			)
 		)
-		(property "Value" "0.33R"
+		(property "Value" "0.33R 1%"
 			(at 166.876 152.18 0)
 			(show_name no)
@@
 			(at 165.1 151.13 0)
 			(hide yes)
+			(show_name no)
+			(do_not_autoplace no)
+			(effects
+				(font
+					(size 1.27 1.27)
+				)
+			)
+		)
+		(property "MPN" "ERJ-6RQFR33V"
+			(at 165.1 151.13 0)
+			(hide yes)
+			(show_name no)
+			(do_not_autoplace no)
+			(effects
+				(font
+					(size 1.27 1.27)
+				)
+			)
+		)
+		(property "Manufacturer" "Panasonic"
+			(at 165.1 151.13 0)
+			(hide yes)
