File: hardware/kicad/rail_monitor.kicad_sch (KiCad schematic)
At the start: 18 parts, among them U14 MCP6569-E/SL

Commit message: feat(hardware): draw decisions D-95, D-97 and D-98
The three decisions that follow the circuit simulations and need no
copper are drawn in the schematic and on the board as changes of
values, part numbers, fitted flags and texts:

- D-95: C32, C33 and C34 of the rail monitor are 10 nF C0G
  (GRM1885C1H103JA01D), not 1 nF.
- D-98: the damper on the input from the controller module is fitted,
  R14 at 0.33 ohm (ERJ-6RQFR33V) and C5 at 10 uF (CL21A106KAYNNNE).
- D-97: the position U9 stays without a part, and its text no longer
  names the detector with the time-out of 0.24 s.

No track, via, zone or footprint position changed. The electrical
rules check and the design rules check with schematic parity report
nothing. The bill of materials (151 lines for 370 parts), the
schematic PDF, the pictures of the three sheets and the two renderings
of the board are exported again.

D-96, the position for a capacitor at U28, is not drawn: it needs a
footprint and copper.
Parts:
- C32, C33, C34: value 1n 50V C0G -> 10n 50V C0G; MPN C0603C102J5GACTU -> GRM1885C1H103JA01D; Manufacturer KEMET -> Murata
Other:
- note added: "C32, C33 and C34, 10 nF each, keep an edge of PWR_GOOD from moving the thresholds through the pin capacitance of the package: each output pin of U14 is the neighbor of an inverting input (time constants about 0.09 ms, 0.25 ms and 0.36 ms, calculated)."
- note removed: "C32, C33 and C34 keep an edge of PWR_GOOD from moving the thresholds through the pin capacitance of the package: each output pin of U14 is the neighbor of an inverting input (time constants 9 us, 25 us and 36 us, calculated)."
Changed lines of the file:
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@@
 		)
 	)
-	(text "C32, C33 and C34 keep an edge of PWR_GOOD from moving the thresholds through\nthe pin capacitance of the package: each output pin of U14 is the neighbor of\nan inverting input (time constants 9 us, 25 us and 36 us, calculated)."
+	(text "C32, C33 and C34, 10 nF each, keep an edge of PWR_GOOD from moving the thresholds\nthrough the pin capacitance of the package: each output pin of U14 is the neighbor\nof an inverting input (time constants about 0.09 ms, 0.25 ms and 0.36 ms, calculated)."
 		(exclude_from_sim no)
 		(at 20.32 163.83 0)
@@
 			)
 		)
-		(property "Value" "1n 50V C0G"
+		(property "Value" "10n 50V C0G"
 			(at 155.192 102.65 0)
 			(show_name no)
@@
 			)
 		)
-		(property "MPN" "C0603C102J5GACTU"
+		(property "MPN" "GRM1885C1H103JA01D"
 			(at 152.4 101.6 0)
 			(hide yes)
@@
 			)
 		)
-		(property "Manufacturer" "KEMET"
+		(property "Manufacturer" "Murata"
 			(at 152.4 101.6 0)
 			(hide yes)
@@
 			)
 		)
-		(property "Value" "1n 50V C0G"
+		(property "Value" "10n 50V C0G"
 			(at 48.512 126.78 0)
 			(show_name no)
@@
 			)
 		)
-		(property "MPN" "C0603C102J5GACTU"
+		(property "MPN" "GRM1885C1H103JA01D"
 			(at 45.72 125.73 0)
 			(hide yes)
@@
 			)
 		)
-		(property "Manufacturer" "KEMET"
+		(property "Manufacturer" "Murata"
 			(at 45.72 125.73 0)
 			(hide yes)
@@
 			)
 		)
-		(property "Value" "1n 50V C0G"
+		(property "Value" "10n 50V C0G"
 			(at 86.612 126.78 0)
 			(show_name no)
@@
 			)
 		)
-		(property "MPN" "C0603C102J5GACTU"
+		(property "MPN" "GRM1885C1H103JA01D"
 			(at 83.82 125.73 0)
 			(hide yes)
@@
 			)
 		)
-		(property "Manufacturer" "KEMET"
+		(property "Manufacturer" "Murata"
 			(at 83.82 125.73 0)
 			(hide yes)
