File: hardware/kicad/power-profiler-carrier.kicad_pcb (KiCad board)
At the start: 4 copper layers, 150 x 100 mm, 425 parts, among them J1 Debug UART, J2 USB-C power, J3 DUT, J4 DUT wires, J5 Logic port, Q1 BSS138, Q10 IRLML0030, Q11 IRLML0030, Q12 IRLML0030, Q13 IRLML0030, Q14 CSD17577Q3A, Q15 CSD17577Q3A, Q16 CSD17577Q3A, Q2 BSS138, Q3 BSS138, Q4 CSD17577Q3A, Q5 CSD17577Q3A, Q6 BC847B, Q7 BC847B, Q8 CSD17577Q3A, Q9 CSD17577Q3A, SW1 RESET, U1 Raspberry Pi Pico 2, U10 LMR62014XMF, U11 LM27761DSG, U12 REF5025AID, U13 LT3042EMSE, U14 MCP6569-E/SL, U15 MCP4921-E/SN, U16 TPS63020DSJ, U17 OPA197IDBV, U18 LT3080EDD, U19 OPA365AIDBV, U2 TPD4E1U06DBVR, U20 TC4427EOA, U21 MCP6561T-E/OT, U22 TC4427EOA, U23 TC4427EOA, U24 MUX509IPWR, U25 OPA197IDBV, U26 OPA197IDBV, U27 AD8421ARZ, U28 OPA365AIDBV, U29 OPA365AIDBV, U3 TPS259621DDAR, U30 ADS8860IDGS, U31 MCP6562-E/SN, U32 MCP6561T-E/OT, U33 SN74LV165ADR, U34 SN74LV165ADR, U35 TPD4E1U06DBVR, U36 TPD4E1U06DBVR, U37 TPD4E1U06DBVR, U38 SN74LVC8T245PW, U39 MCP9700AT-E/TT, U4 TPS259621DDAR, U40 MCP3208-BI/SL, U5 TPS2116DRLR, U6 TPS3808G01DBVR, U7 LP5907MFX-3.3, U8 LP5907MFX-3.3, U9 803 type, 3.08 V

Commit message: feat(hardware): draw decisions D-95, D-97 and D-98
The three decisions that follow the circuit simulations and need no
copper are drawn in the schematic and on the board as changes of
values, part numbers, fitted flags and texts:

- D-95: C32, C33 and C34 of the rail monitor are 10 nF C0G
  (GRM1885C1H103JA01D), not 1 nF.
- D-98: the damper on the input from the controller module is fitted,
  R14 at 0.33 ohm (ERJ-6RQFR33V) and C5 at 10 uF (CL21A106KAYNNNE).
- D-97: the position U9 stays without a part, and its text no longer
  names the detector with the time-out of 0.24 s.

No track, via, zone or footprint position changed. The electrical
rules check and the design rules check with schematic parity report
nothing. The bill of materials (151 lines for 370 parts), the
schematic PDF, the pictures of the three sheets and the two renderings
of the board are exported again.

D-96, the position for a capacitor at U28, is not drawn: it needs a
footprint and copper.
Parts:
- C32, C33, C34: value 1n 50V C0G -> 10n 50V C0G
- C5: value 10u 25V -> 10u 25V X5R
- R14: value 0.33R -> 0.33R 1%
- U9: value 803 type, 3.08 V -> Detector, ms time-out
Changed lines of the file:
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@@
 			)
 		)
-		(property "Value" "1n 50V C0G"
+		(property "Value" "10n 50V C0G"
 			(at 0 1.43 180)
 			(layer "F.Fab")
@@
 			)
 		)
-		(property "MPN" "C0603C102J5GACTU"
+		(property "MPN" "GRM1885C1H103JA01D"
 			(at 0 0 180)
 			(layer "F.Fab")
@@
 			)
 		)
-		(property "Manufacturer" "KEMET"
+		(property "Manufacturer" "Murata"
 			(at 0 0 180)
 			(layer "F.Fab")
@@
 			)
 		)
-		(property "Value" "803 type, 3.08 V"
+		(property "Value" "Detector, ms time-out"
 			(at 0 2.4 90)
 			(layer "F.Fab")
@@
 			)
 		)
-		(property "Value" "0.33R"
+		(property "Value" "0.33R 1%"
 			(at 0 1.65 0)
 			(layer "F.Fab")
@@
 			)
 		)
+		(property "MPN" "ERJ-6RQFR33V"
+			(at 0 0 0)
+			(layer "F.Fab")
+			(hide yes)
+			(effects
+				(font
+					(size 1.27 1.27)
+					(thickness 0.15)
+				)
+			)
+		)
+		(property "Manufacturer" "Panasonic"
+			(at 0 0 0)
+			(layer "F.Fab")
+			(hide yes)
+			(effects
+				(font
+					(size 1.27 1.27)
+					(thickness 0.15)
+				)
+			)
+		)
 		(property ki_fp_filters "R_*")
 		(sheetname "/Power Input/")
@@
 			)
 		)
-		(attr smd exclude_from_bom dnp)
+		(attr smd)
 		(duplicate_pad_numbers_are_jumpers no)
 		(fp_line
@@
 			)
 		)
-		(property "Value" "1n 50V C0G"
+		(property "Value" "10n 50V C0G"
 			(at 0 1.43 180)
 			(layer "F.Fab")
@@
 			)
 		)
-		(property "MPN" "C0603C102J5GACTU"
+		(property "MPN" "GRM1885C1H103JA01D"
 			(at 0 0 180)
 			(layer "F.Fab")
@@
 			)
 		)
-		(property "Manufacturer" "KEMET"
+		(property "Manufacturer" "Murata"
 			(at 0 0 180)
 			(layer "F.Fab")
@@
 			)
 		)
-		(property "Value" "10u 25V"
+		(property "Value" "10u 25V X5R"
 			(at 0 1.68 270)
 			(layer "F.Fab")
@@
 			)
 		)
+		(property "MPN" "CL21A106KAYNNNE"
+			(at 0 0 270)
+			(layer "F.Fab")
+			(hide yes)
+			(effects
+				(font
+					(size 1.27 1.27)
+					(thickness 0.15)
+				)
+			)
+		)
+		(property "Manufacturer" "Samsung Electro-Mechanics"
+			(at 0 0 270)
+			(layer "F.Fab")
+			(hide yes)
+			(effects
+				(font
+					(size 1.27 1.27)
+					(thickness 0.15)
+				)
+			)
+		)
 		(property ki_fp_filters "C_*")
 		(sheetname "/Power Input/")
@@
 			)
 		)
-		(attr smd exclude_from_bom dnp)
+		(attr smd)
 		(duplicate_pad_numbers_are_jumpers no)
 		(fp_line
@@
 			)
 		)
-		(property "Value" "1n 50V C0G"
+		(property "Value" "10n 50V C0G"
 			(at 0 1.43 270)
 			(layer "F.Fab")
@@
 			)
 		)
-		(property "MPN" "C0603C102J5GACTU"
+		(property "MPN" "GRM1885C1H103JA01D"
 			(at 0 0 270)
 			(layer "F.Fab")
@@
 			)
 		)
-		(property "Manufacturer" "KEMET"
+		(property "Manufacturer" "Murata"
 			(at 0 0 270)
 			(layer "F.Fab")

Commit message: fix(hardware): apply review findings and frame the blocks on silk
The review of footprints and placement of 2026-10-13 found five
points on the carrier board (draft A2). This commit corrects them and
adds the frames of the placement blocks to the silkscreen. Nothing
was routed again: every track, 683 of the 694 vias, the place of
every footprint and the outline of every copper zone are unchanged.

- U16 (TPS63020DSJR) stood on the land pattern of another maker's
  package of the same body. It has the land pattern of the TI DSJ
  package now, a new project footprint: thermal land 1.58 mm x
  2.85 mm, lands 0.60 mm x 0.24 mm, eight paste openings. The sheet,
  the project symbol and one line of the bill of materials name it.
- Eleven vias moved by 0.2 mm to 1.6 mm, each joined to its old place
  by a short piece of track (27 pieces, 15.9 mm in all): nine whose
  hole stood in a pad or within 0.05 mm of one, and two that stood
  under the wall line of the shield can.
- Silkscreen: the frames and names of the sixteen placement blocks,
  cut where a pad, a mask opening, a part or a text is in the way;
  TX, RX and GND at J1; "PICO USB" over "DATA/POWER"; 61 reference
  texts moved to their own part, 31 hidden ones shown again, three
  hidden. 330 are visible and 95 hidden, where it was 302 and 123.
- The frames and names of the blocks were on the layer User.Drawings
  and are removed there.

Checked with KiCad 10.0.0: electrical rules check 0 messages; design
rules check with schematic parity 0 violations, 0 unconnected pads,
0 footprint errors. The calculated figures of the board are the same
as before: 19.5 and 23.3 squares on the 1 A path, 5.1 nA of surface
leakage into the measured node.
Parts:
- U16: footprint Package_DFN_QFN:DFN-14-1EP_3x4mm_P0.5mm_EP1.7x3.3mm -> PowerProfiler:Texas_R-PVSON-N14_3x4mm_P0.5mm_EP1.58x2.85mm
Routing:
- net Net-(Q1-S): track 21.5 -> 26.6 mm
- net +3V3_A: track 365.2 -> 366.9 mm
- net /Controller/PWR_GOOD: track 202.9 -> 204.5 mm
- net Net-(U26--): track 43.1 -> 44.6 mm
- net VREF: track 538.3 -> 539.7 mm
- net /Controller/GATE_SRC: track 123.0 -> 124.1 mm
- net /Comparators/AMP_RAW: track 70.7 -> 71.8 mm
- net Net-(D17-A): track 36.4 -> 37.4 mm
- net Net-(U14B--): track 7.42 -> 8.27 mm
- net GND: track 302.4 -> 303.2 mm
Other:
- board text added: "DATA/POWER"
- board text added: "PICO USB"
- board text added: "RX"
- board text added: "TX"
- board text removed: "USB DATA/POWER"
