File: hardware/kicad/source_meter.kicad_sch (KiCad schematic)
At the start: 58 parts, among them Q1 BSS138, U15 MCP4921-E/SN, U16 TPS63020DSJ, U17 OPA197IDBV, U18 LT3080EDD, U19 OPA365AIDBV

Commit message: fix(hardware): apply review findings and frame the blocks on silk
The review of footprints and placement of 2026-10-13 found five
points on the carrier board (draft A2). This commit corrects them and
adds the frames of the placement blocks to the silkscreen. Nothing
was routed again: every track, 683 of the 694 vias, the place of
every footprint and the outline of every copper zone are unchanged.

- U16 (TPS63020DSJR) stood on the land pattern of another maker's
  package of the same body. It has the land pattern of the TI DSJ
  package now, a new project footprint: thermal land 1.58 mm x
  2.85 mm, lands 0.60 mm x 0.24 mm, eight paste openings. The sheet,
  the project symbol and one line of the bill of materials name it.
- Eleven vias moved by 0.2 mm to 1.6 mm, each joined to its old place
  by a short piece of track (27 pieces, 15.9 mm in all): nine whose
  hole stood in a pad or within 0.05 mm of one, and two that stood
  under the wall line of the shield can.
- Silkscreen: the frames and names of the sixteen placement blocks,
  cut where a pad, a mask opening, a part or a text is in the way;
  TX, RX and GND at J1; "PICO USB" over "DATA/POWER"; 61 reference
  texts moved to their own part, 31 hidden ones shown again, three
  hidden. 330 are visible and 95 hidden, where it was 302 and 123.
- The frames and names of the blocks were on the layer User.Drawings
  and are removed there.

Checked with KiCad 10.0.0: electrical rules check 0 messages; design
rules check with schematic parity 0 violations, 0 unconnected pads,
0 footprint errors. The calculated figures of the board are the same
as before: 19.5 and 23.3 squares on the 1 A path, 5.1 nA of surface
leakage into the measured node.
Parts:
- U16: footprint Package_DFN_QFN:DFN-14-1EP_3x4mm_P0.5mm_EP1.7x3.3mm -> PowerProfiler:Texas_R-PVSON-N14_3x4mm_P0.5mm_EP1.58x2.85mm
Changed lines of the file:
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@@
 			)
 		)
-		(property "Footprint" "Package_DFN_QFN:DFN-14-1EP_3x4mm_P0.5mm_EP1.7x3.3mm"
+		(property "Footprint" "PowerProfiler:Texas_R-PVSON-N14_3x4mm_P0.5mm_EP1.58x2.85mm"
 			(at 83.82 48.26 0)
 			(hide yes)
